File: pcb/right/interphase.sch (KiCad schematic (older format))
At the start: 75 parts, among them J1 Conn_01x04_Male, SW10 MOM-SPST, SW11 MOM-SPST, SW12 MOM-SPST, SW13 MOM-SPST, SW14 MOM-SPST, SW15 MOM-SPST, SW16 MOM-SPST, SW17 MOM-SPST, SW18 MOM-SPST, SW19 MOM-SPST, SW2 MOM-SPST, SW20 MOM-SPST, SW21 MOM-SPST, SW22 MOM-SPST, SW23 MOM-SPST, SW24 MOM-SPST, SW25 MOM-SPST, SW27 MOM-SPST, SW28 MOM-SPST, SW29 MOM-SPST, SW3 MOM-SPST, SW30 MOM-SPST, SW32 MOM-SPST, SW33 MOM-SPST, SW34 MOM-SPST, SW37 MOM-SPST, SW38 MOM-SPST, SW4 MOM-SPST, SW5 MOM-SPST, SW6 MOM-SPST, SW7 MOM-SPST, SW8 MOM-SPST, SW9 MOM-SPST, U1 Core51822B, U2 MCP1640

Commit message: add tmk support
Parts:
- removed C1: 4,7µF, Capacitors_SMD:C_0805_HandSoldering, symbol C-RESCUE-interphase
- removed C2: 10µF, Capacitors_SMD:C_0805_HandSoldering, symbol C-RESCUE-interphase
- removed L1: 4,7µH, SMD_Packages:SMD-1206_Pol, symbol L
- removed R1: 536K, Resistors_SMD:R_0805, symbol R-RESCUE-interphase
- removed R2: 309K, Resistors_SMD:R_0805, symbol R-RESCUE-interphase
- removed U2: MCP1640, TO_SOT_Packages_SMD:SOT-23-6, symbol MCP1640
- added SW1: SW_SPDT, Button_Switch_Keyboard:SW_E-Switch_EG1224_SPDT, symbol SW_SPDT
Connections:
- net labels removed: +BATT
- wire segments 122 -> 110
Changed lines of the file:
@@
-$EndComp
-$Comp
-L MCP1640 U2
-U 1 1 59BFA9D7
-P 2350 5400
-F 0 "U2" H 2450 5800 60  0000 C CNN
-F 1 "MCP1640" H 2550 4950 60  0000 C CNN
-F 2 "TO_SOT_Packages_SMD:SOT-23-6" H 2350 5400 60  0001 C CNN
-F 3 "" H 2350 5400 60  0001 C CNN
-	1    2350 5400
-	1    0    0    -1
-$EndComp
-$Comp
-L C-RESCUE-interphase C1
-U 1 1 59BFAAF6
-P 1450 5550
-F 0 "C1" H 1475 5650 50  0000 L CNN
-F 1 "4,7µF" H 1475 5450 50  0000 L CNN
-F 2 "Capacitors_SMD:C_0805_HandSoldering" H 1488 5400 50  0001 C CNN
-F 3 "" H 1450 5550 50  0001 C CNN
-	1    1450 5550
-	1    0    0    -1
-$EndComp
-$Comp
-L L L1
-U 1 1 59BFAB7F
-P 1800 4900
-F 0 "L1" V 1750 4900 50  0000 C CNN
-F 1 "4,7µH" V 1875 4900 50  0000 C CNN
-F 2 "SMD_Packages:SMD-1206_Pol" H 1800 4900 50  0001 C CNN
-F 3 "" H 1800 4900 50  0001 C CNN
-	1    1800 4900
-	0    -1   -1   0
-$EndComp
-$Comp
-L R-RESCUE-interphase R1
-U 1 1 59BFABC2
-P 2950 5250
-F 0 "R1" V 3030 5250 50  0000 C CNN
-F 1 "536K" V 2950 5250 50  0000 C CNN
-F 2 "Resistors_SMD:R_0805" V 2880 5250 50  0001 C CNN
-F 3 "" H 2950 5250 50  0001 C CNN
-	1    2950 5250
-	1    0    0    -1
-$EndComp
-$Comp
-L R-RESCUE-interphase R2
-U 1 1 59BFAC0F
-P 2950 5650
-F 0 "R2" V 3030 5650 50  0000 C CNN
-F 1 "309K" V 2950 5650 50  0000 C CNN
-F 2 "Resistors_SMD:R_0805" V 2880 5650 50  0001 C CNN
-F 3 "" H 2950 5650 50  0001 C CNN
-	1    2950 5650
-	1    0    0    -1
-$EndComp
-$Comp
-L C-RESCUE-interphase C2
-U 1 1 59BFAC64
-P 3350 5450
-F 0 "C2" H 3375 5550 50  0000 L CNN
-F 1 "10µF" H 3375 5350 50  0000 L CNN
-F 2 "Capacitors_SMD:C_0805_HandSoldering" H 3388 5300 50  0001 C CNN
-F 3 "" H 3350 5450 50  0001 C CNN
-	1    3350 5450
-	1    0    0    -1
 $EndComp
 $Comp
@@
 $EndComp
 $Comp
-L +3.3V #PWR02
-U 1 1 59C15857
-P 3350 4900
-F 0 "#PWR02" H 3350 4750 50  0001 C CNN
-F 1 "+3.3V" H 3350 5040 50  0000 C CNN
-F 2 "" H 3350 4900 50  0001 C CNN
-F 3 "" H 3350 4900 50  0001 C CNN
-	1    3350 4900
-	1    0    0    -1
-$EndComp
-$Comp
-L GND #PWR03
+L GND #PWR02
 U 1 1 59C23F89
-P 3750 2300
-F 0 "#PWR03" H 3750 2050 50  0001 C CNN
-F 1 "GND" H 3750 2150 50  0000 C CNN
-F 2 "" H 3750 2300 50  0001 C CNN
-F 3 "" H 3750 2300 50  0001 C CNN
-	1    3750 2300
-	1    0    0    -1
+P 3550 1700
+F 0 "#PWR02" H 3550 1450 50  0001 C CNN
+F 1 "GND" H 3550 1550 50  0000 C CNN
+F 2 "" H 3550 1700 50  0001 C CNN
+F 3 "" H 3550 1700 50  0001 C CNN
+	1    3550 1700
+	0    -1   -1   0
 $EndComp
 $Comp
@@
 $EndComp
 $Comp
-L +3.3V #PWR04
+L +3.3V #PWR03
 U 1 1 59CC64DF
 P 3750 1250
-F 0 "#PWR04" H 3750 1100 50  0001 C CNN
+F 0 "#PWR03" H 3750 1100 50  0001 C CNN
 F 1 "+3.3V" H 3750 1390 50  0000 C CNN
 F 2 "" H 3750 1250 50  0001 C CNN
@@
 $EndComp
 $Comp
-L GND #PWR05
+L GND #PWR04
 U 1 1 59CC64E5
 P 4300 5750
-F 0 "#PWR05" H 4300 5500 50  0001 C CNN
+F 0 "#PWR04" H 4300 5500 50  0001 C CNN
 F 1 "GND" H 4300 5600 50  0000 C CNN
 F 2 "" H 4300 5750 50  0001 C CNN
@@
 $EndComp
 $Comp
-L +BATT #PWR06
-U 1 1 59CD076E
-P 5050 6150
-F 0 "#PWR06" H 5050 6000 50  0001 C CNN
-F 1 "+BATT" H 5050 6290 50  0000 C CNN
-F 2 "" H 5050 6150 50  0001 C CNN
-F 3 "" H 5050 6150 50  0001 C CNN
-	1    5050 6150
-	1    0    0    -1
-$EndComp
-$Comp
-L +BATT #PWR07
-U 1 1 59CD0834
-P 1050 4950
-F 0 "#PWR07" H 1050 4800 50  0001 C CNN
-F 1 "+BATT" H 1050 5090 50  0000 C CNN
-F 2 "" H 1050 4950 50  0001 C CNN
-F 3 "" H 1050 4950 50  0001 C CNN
-	1    1050 4950
-	1    0    0    -1
-$EndComp
-$Comp
-L +3.3V #PWR08
+L +3.3V #PWR05
 U 1 1 59CFE3BD
 P 5850 5050
-F 0 "#PWR08" H 5850 4900 50  0001 C CNN
+F 0 "#PWR05" H 5850 4900 50  0001 C CNN
 F 1 "+3.3V" H 5850 5190 50  0000 C CNN
 F 2 "" H 5850 5050 50  0001 C CNN
@@
 	1    0    0    -1
 $EndComp
-$Comp
-L GND #PWR09
-U 1 1 59BBF383
-P 1500 6050
-F 0 "#PWR09" H 1500 5800 50  0001 C CNN
-F 1 "GND" H 1500 5900 50  0000 C CNN
-F 2 "" H 1500 6050 50  0001 C CNN
-F 3 "" H 1500 6050 50  0001 C CNN
-	1    1500 6050
-	1    0    0    -1
-$EndComp
 Wire Wire Line
 	700  5400 700  5300
 Wire Wire Line
-	700  5300 1900 5300
-Wire Wire Line
-	1450 5400 1450 5300
-Connection ~ 1450 5300
-Wire Wire Line
 	1650 4900 1550 4900
-Wire Wire Line
-	1550 4900 1550 5300
 Connection ~ 1550 5300
 Wire Wire Line
@@
 	2950 5100 2950 5050
 Connection ~ 2950 5050
-Wire Wire Line
-	1500 5900 1500 6050
-Wire Wire Line
-	700  5900 3350 5900
-Connection ~ 1500 5900
-Wire Wire Line
-	1450 5700 1450 5900
-Connection ~ 1450 5900
 Wire Wire Line
 	2950 5900 2950 5800
@@
 Connection ~ 8300 1550
 Connection ~ 700  5900
-Connection ~ 1050 5300
 Wire Wire Line
 	5200 6150 5050 6150
 Connection ~ 5200 6150
 Wire Wire Line
-	1050 4950 1050 5300
-Wire Wire Line
-	5200 5650 5200 6150
-Wire Wire Line
-	4050 3200 4700 3200
+	3750 3200 4700 3200
 Wire Wire Line
 	4700 3200 4700 3250
@@
 Wire Wire Line
 	3750 1600 3750 1250
-Wire Wire Line
-	3550 1700 4050 1700
 Wire Wire Line
 	3550 1800 4000 1800
@@
 	5300 5550 4300 5550
 Wire Wire Line
-	5200 5650 6000 5650
-Wire Wire Line
-	6000 5650 6000 4550
-Wire Wire Line
 	6000 4550 5850 4550
 Wire Wire Line
 	3550 1900 3750 1900
 Wire Wire Line
-	3750 1900 3750 2300
+	3750 1900 3750 3200
 Connection ~ 4300 5550
 Connection ~ 4000 1800
@@
 Wire Wire Line
 	6500 950  6500 3700
-Connection ~ 1150 5300
 Wire Wire Line
 	700  5700 700  5900
 Wire Wire Line
 	4000 1800 4000 3150
-Wire Wire Line
-	4050 1700 4050 3200
 Text Label 5650 650  0    60   ~ 0
 row0
@@
 	6000 3350 6000 3050
 Connection ~ 6000 3050
+$Comp
+L SW_SPDT SW1
+U 1 1 5ADEA364
+P 800 5100
+F 0 "SW1" H 800 5270 50  0000 C CNN
+F 1 "SW_SPDT" H 800 4900 50  0000 C CNN
+F 2 "Button_Switch_Keyboard:SW_E-Switch_EG1224_SPDT" H 800 5100 50  0001 C CNN
+F 3 "" H 800 5100 50  0001 C CNN
+	1    800  5100
+	0    1    1    0
+$EndComp
+$Comp
+L +3.3V #PWR06
+U 1 1 59C15857
+P 800 4900
+F 0 "#PWR06" H 800 4750 50  0001 C CNN
+F 1 "+3.3V" H 800 5040 50  0000 C CNN
+F 2 "" H 800 4900 50  0001 C CNN
+F 3 "" H 800 4900 50  0001 C CNN
+	1    800  4900
+	1    0    0    -1
+$EndComp
+$Comp
+L GND #PWR?
+U 1 1 5ADEC7F1
+P 700 5900
+F 0 "#PWR?" H 700 5650 50  0001 C CNN
+F 1 "GND" H 700 5750 50  0000 C CNN
+F 2 "" H 700 5900 50  0001 C CNN
+F 3 "" H 700 5900 50  0001 C CNN
+	1    700  5900
+	1    0    0    -1
+$EndComp
 $EndSCHEMATC
