File: pcb/right/interphase.kicad_pcb (KiCad board)
At the start: 2 copper layers, 161.9 x 95.3 mm, 75 parts, among them J1 Conn_01x04_Male, SW10 MOM-SPST, SW11 MOM-SPST, SW12 MOM-SPST, SW13 MOM-SPST, SW14 MOM-SPST, SW15 MOM-SPST, SW16 MOM-SPST, SW17 MOM-SPST, SW18 MOM-SPST, SW19 MOM-SPST, SW2 MOM-SPST, SW20 MOM-SPST, SW21 MOM-SPST, SW22 MOM-SPST, SW23 MOM-SPST, SW24 MOM-SPST, SW25 MOM-SPST, SW27 MOM-SPST, SW28 MOM-SPST, SW29 MOM-SPST, SW3 MOM-SPST, SW30 MOM-SPST, SW32 MOM-SPST, SW33 MOM-SPST, SW34 MOM-SPST, SW37 MOM-SPST, SW38 MOM-SPST, SW4 MOM-SPST, SW5 MOM-SPST, SW6 MOM-SPST, SW7 MOM-SPST, SW8 MOM-SPST, SW9 MOM-SPST, U1 Core51822B, U2 MCP1640

Commit message: add tmk support
Parts:
- removed C1: 4,7µF, Capacitors_SMD:C_0805_HandSoldering
- removed C2: 10µF, Capacitors_SMD:C_0805_HandSoldering
- removed L1: 4,7µH, SMD_Packages:SMD-1206_Pol
- removed R1: 536K, Resistors_SMD:R_0805
- removed R2: 309K, Resistors_SMD:R_0805
- removed U2: MCP1640, TO_SOT_Packages_SMD:SOT-23-6
- added SW1: SW_SPDT, Button_Switch_Keyboard:SW_E-Switch_EG1224_SPDT_Angled, F.Cu at (143.0, 90.0)
- moved J1 47.0 mm to (129.9, 92.9), turned to 270 degrees
Connections:
- BT1 pad 1: +BATT -> Net-(BT1-Pad1)
- J1 pad 2: Net-(J1-Pad2) -> GND
- J1 pad 4: GND -> Net-(J1-Pad4)
- U1 pad 15: +BATT -> Net-(U1-Pad15)
- U1 pad 32: Net-(J1-Pad2) -> Net-(J1-Pad4)
Routing:
- net +BATT: track 76.5 -> 0.00 mm, vias 5 -> 0
- net Net-(J1-Pad4): track 0.00 -> 33.9 mm, vias 0 -> 2
- net Net-(BT1-Pad1): track 0.00 -> 26.5 mm, vias 0 -> 3
- net GND: track 135.5 -> 112.0 mm, vias 2 -> 5
- net Net-(J1-Pad2): track 14.9 -> 0.00 mm
- net Net-(J1-Pad3): track 25.8 -> 39.4 mm, vias 0 -> 2
- net Net-(L1-Pad2): track 8.19 -> 0.00 mm
- net Net-(R1-Pad2): track 5.44 -> 0.00 mm
- net /row4: track 138.9 -> 142.8 mm
- net +3V3: track 59.8 -> 57.0 mm, vias 4 -> 1

Commit message: change to actual matrix
Parts:
- moved D36 12.8 mm to (173.2, 35.9)
- moved D21 12.7 mm to (115.9, 35.9)
- moved D31 12.7 mm to (154.0, 35.9)
- moved D11 12.6 mm to (77.8, 35.8)
- moved D26 12.6 mm to (134.9, 35.8)
- moved D16 12.6 mm to (96.8, 35.8)
- moved D12 12.6 mm to (68.5, 54.7)
- moved D7 12.5 mm to (49.3, 54.7)
- moved D6 12.5 mm to (58.8, 35.6)
- moved D27 12.3 mm to (125.4, 54.5)
- moved D32 12.2 mm to (144.3, 54.5)
- moved D22 12.2 mm to (106.5, 54.3)
- moved D37 12.1 mm to (168.2, 54.3)
- moved D17 12.0 mm to (87.3, 54.2)
- moved D20 9.04 mm to (101.7, 92.8), turned to 180 degrees
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Routing:
- net /col3: track 147.7 -> 130.7 mm
- net /col5: track 117.0 -> 102.0 mm
- net Net-(D20-Pad2): track 5.51 -> 20.5 mm
- net /col4: track 126.7 -> 112.3 mm
- net /row4: track 142.8 -> 131.0 mm, vias 1 -> 2
- net /col6: track 106.6 -> 97.7 mm
- net /col2: track 177.9 -> 169.8 mm
- net Net-(D5-Pad2): track 5.32 -> 13.0 mm
- net Net-(D10-Pad2): track 5.51 -> 12.9 mm
- net Net-(D15-Pad2): track 5.51 -> 12.4 mm
- net +3V3: track 57.0 -> 63.7 mm, vias 1 -> 3
- net GND: track 112.0 -> 118.5 mm, vias 5 -> 7
- net /col1: track 200.0 -> 194.2 mm
- net /col7: track 94.8 -> 89.7 mm
- net /col0: track 214.2 -> 217.9 mm
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Other:
- outline, holes or cut-outs redrawn
