File: pcb/left/interphase.sch (KiCad schematic (older format))
At the start: 69 parts, among them J1 Conn_01x04_Male, SW10 MOM-SPST, SW11 MOM-SPST, SW12 MOM-SPST, SW13 MOM-SPST, SW14 MOM-SPST, SW15 MOM-SPST, SW16 MOM-SPST, SW17 MOM-SPST, SW18 MOM-SPST, SW19 MOM-SPST, SW2 MOM-SPST, SW20 MOM-SPST, SW21 MOM-SPST, SW22 MOM-SPST, SW23 MOM-SPST, SW24 MOM-SPST, SW25 MOM-SPST, SW26 MOM-SPST, SW27 MOM-SPST, SW28 MOM-SPST, SW29 MOM-SPST, SW3 MOM-SPST, SW30 MOM-SPST, SW31 MOM-SPST, SW32 MOM-SPST, SW4 MOM-SPST, SW5 MOM-SPST, SW7 MOM-SPST, SW8 MOM-SPST, SW9 MOM-SPST, U1 Core51822B, U2 MCP1640

Commit message: change pcb
Connections:
- wire segments 116 -> 110
Changed lines of the file:
@@
 LIBS:switches
 LIBS:mcp1640
-LIBS:interphase-cache
 EELAYER 25 0
 EELAYER END
@@
 L GND #PWR03
 U 1 1 59C23F89
-P 3750 2300
-F 0 "#PWR03" H 3750 2050 50  0001 C CNN
-F 1 "GND" H 3750 2150 50  0000 C CNN
-F 2 "" H 3750 2300 50  0001 C CNN
-F 3 "" H 3750 2300 50  0001 C CNN
-	1    3750 2300
-	1    0    0    -1
+P 3550 1700
+F 0 "#PWR03" H 3550 1450 50  0001 C CNN
+F 1 "GND" H 3550 1550 50  0000 C CNN
+F 2 "" H 3550 1700 50  0001 C CNN
+F 3 "" H 3550 1700 50  0001 C CNN
+	1    3550 1700
+	0    -1   -1   0
 $EndComp
 $Comp
@@
 	5200 5650 5200 6150
 Wire Wire Line
-	4050 3200 4700 3200
-Wire Wire Line
-	4700 3200 4700 3250
-Wire Wire Line
-	4000 3150 4800 3150
-Wire Wire Line
-	4800 3150 4800 3250
+	4700 1900 4700 3250
+Wire Wire Line
+	4800 1800 4800 3250
 Wire Wire Line
 	3550 1600 3750 1600
@@
 	3750 1600 3750 1250
 Wire Wire Line
-	3550 1700 4050 1700
-Wire Wire Line
-	3550 1800 4000 1800
-Wire Wire Line
 	4800 800  4800 900
 Wire Wire Line
@@
 Wire Wire Line
 	5850 5150 5850 5050
-Connection ~ 3750 2250
 Wire Wire Line
 	4300 5150 4300 5750
@@
 Wire Wire Line
 	6000 4550 5850 4550
-Wire Wire Line
-	3550 1900 3750 1900
-Wire Wire Line
-	3750 1900 3750 2300
 Connection ~ 4300 5550
-Connection ~ 4000 1800
-Connection ~ 4050 1700
 Wire Wire Line
 	11050 950  11050 4300
@@
 Wire Wire Line
 	700  5700 700  5900
-Wire Wire Line
-	4000 1800 4000 3150
-Wire Wire Line
-	4050 1700 4050 3200
 $Comp
 L D-RESCUE-interphase D30
@@
 Wire Wire Line
 	9950 3050 6650 3050
+Wire Wire Line
+	3550 1800 4800 1800
+Wire Wire Line
+	3550 1900 4700 1900
 $EndSCHEMATC

Commit message: can send basic chars
Parts:
- removed C1: 4,7µF, Capacitors_SMD:C_0805_HandSoldering, symbol C-RESCUE-interphase
- removed C2: 10µF, Capacitors_SMD:C_0805_HandSoldering, symbol C-RESCUE-interphase
- removed L1: 4,7µH, SMD_Packages:SMD-1206_Pol, symbol L
- removed R1: 536K, Resistors_SMD:R_0805, symbol R-RESCUE-interphase
- removed R2: 309K, Resistors_SMD:R_0805, symbol R-RESCUE-interphase
- removed U2: MCP1640, TO_SOT_Packages_SMD:SOT-23-6, symbol MCP1640
Connections:
- wire segments 110 -> 101
Changed lines of the file:
@@
-$EndComp
-$Comp
-L MCP1640 U2
-U 1 1 59BFA9D7
-P 2350 5400
-F 0 "U2" H 2450 5800 60  0000 C CNN
-F 1 "MCP1640" H 2550 4950 60  0000 C CNN
-F 2 "TO_SOT_Packages_SMD:SOT-23-6" H 2350 5400 60  0001 C CNN
-F 3 "" H 2350 5400 60  0001 C CNN
-	1    2350 5400
-	1    0    0    -1
-$EndComp
-$Comp
-L C-RESCUE-interphase C1
-U 1 1 59BFAAF6
-P 1450 5550
-F 0 "C1" H 1475 5650 50  0000 L CNN
-F 1 "4,7µF" H 1475 5450 50  0000 L CNN
-F 2 "Capacitors_SMD:C_0805_HandSoldering" H 1488 5400 50  0001 C CNN
-F 3 "" H 1450 5550 50  0001 C CNN
-	1    1450 5550
-	1    0    0    -1
-$EndComp
-$Comp
-L L L1
-U 1 1 59BFAB7F
-P 1800 4900
-F 0 "L1" V 1750 4900 50  0000 C CNN
-F 1 "4,7µH" V 1875 4900 50  0000 C CNN
-F 2 "SMD_Packages:SMD-1206_Pol" H 1800 4900 50  0001 C CNN
-F 3 "" H 1800 4900 50  0001 C CNN
-	1    1800 4900
-	0    -1   -1   0
-$EndComp
-$Comp
-L R-RESCUE-interphase R1
-U 1 1 59BFABC2
-P 2950 5250
-F 0 "R1" V 3030 5250 50  0000 C CNN
-F 1 "536K" V 2950 5250 50  0000 C CNN
-F 2 "Resistors_SMD:R_0805" V 2880 5250 50  0001 C CNN
-F 3 "" H 2950 5250 50  0001 C CNN
-	1    2950 5250
-	1    0    0    -1
-$EndComp
-$Comp
-L R-RESCUE-interphase R2
-U 1 1 59BFAC0F
-P 2950 5650
-F 0 "R2" V 3030 5650 50  0000 C CNN
-F 1 "309K" V 2950 5650 50  0000 C CNN
-F 2 "Resistors_SMD:R_0805" V 2880 5650 50  0001 C CNN
-F 3 "" H 2950 5650 50  0001 C CNN
-	1    2950 5650
-	1    0    0    -1
-$EndComp
-$Comp
-L C-RESCUE-interphase C2
-U 1 1 59BFAC64
-P 3350 5450
-F 0 "C2" H 3375 5550 50  0000 L CNN
-F 1 "10µF" H 3375 5350 50  0000 L CNN
-F 2 "Capacitors_SMD:C_0805_HandSoldering" H 3388 5300 50  0001 C CNN
-F 3 "" H 3350 5450 50  0001 C CNN
-	1    3350 5450
-	1    0    0    -1
 $EndComp
 $Comp
@@
 $EndComp
 $Comp
-L +3.3V #PWR02
-U 1 1 59C15857
-P 3350 4900
-F 0 "#PWR02" H 3350 4750 50  0001 C CNN
-F 1 "+3.3V" H 3350 5040 50  0000 C CNN
-F 2 "" H 3350 4900 50  0001 C CNN
-F 3 "" H 3350 4900 50  0001 C CNN
-	1    3350 4900
-	1    0    0    -1
-$EndComp
-$Comp
-L GND #PWR03
+L GND #PWR02
 U 1 1 59C23F89
 P 3550 1700
-F 0 "#PWR03" H 3550 1450 50  0001 C CNN
+F 0 "#PWR02" H 3550 1450 50  0001 C CNN
 F 1 "GND" H 3550 1550 50  0000 C CNN
 F 2 "" H 3550 1700 50  0001 C CNN
@@
 $EndComp
 $Comp
-L +3.3V #PWR04
+L +3.3V #PWR03
 U 1 1 59CC64DF
 P 3750 1250
-F 0 "#PWR04" H 3750 1100 50  0001 C CNN
+F 0 "#PWR03" H 3750 1100 50  0001 C CNN
 F 1 "+3.3V" H 3750 1390 50  0000 C CNN
 F 2 "" H 3750 1250 50  0001 C CNN
@@
 $EndComp
 $Comp
-L GND #PWR05
+L GND #PWR04
 U 1 1 59CC64E5
 P 4300 5750
-F 0 "#PWR05" H 4300 5500 50  0001 C CNN
+F 0 "#PWR04" H 4300 5500 50  0001 C CNN
 F 1 "GND" H 4300 5600 50  0000 C CNN
 F 2 "" H 4300 5750 50  0001 C CNN
@@
 $EndComp
 $Comp
-L +BATT #PWR06
+L +BATT #PWR05
 U 1 1 59CD076E
 P 5050 6150
-F 0 "#PWR06" H 5050 6000 50  0001 C CNN
+F 0 "#PWR05" H 5050 6000 50  0001 C CNN
 F 1 "+BATT" H 5050 6290 50  0000 C CNN
 F 2 "" H 5050 6150 50  0001 C CNN
@@
 $EndComp
 $Comp
-L +BATT #PWR07
-U 1 1 59CD0834
-P 1050 4950
-F 0 "#PWR07" H 1050 4800 50  0001 C CNN
-F 1 "+BATT" H 1050 5090 50  0000 C CNN
-F 2 "" H 1050 4950 50  0001 C CNN
-F 3 "" H 1050 4950 50  0001 C CNN
-	1    1050 4950
-	1    0    0    -1
-$EndComp
-$Comp
-L +3.3V #PWR08
+L +3.3V #PWR06
 U 1 1 59CFE3BD
 P 5850 5050
-F 0 "#PWR08" H 5850 4900 50  0001 C CNN
+F 0 "#PWR06" H 5850 4900 50  0001 C CNN
 F 1 "+3.3V" H 5850 5190 50  0000 C CNN
 F 2 "" H 5850 5050 50  0001 C CNN
@@
 F 5 "Switch" H 9475 3650 40  0001 L BNN "Family"
 	1    9400 3350
-	1    0    0    -1
-$EndComp
-$Comp
-L GND #PWR09
-U 1 1 59BBF383
-P 1500 6050
-F 0 "#PWR09" H 1500 5800 50  0001 C CNN
-F 1 "GND" H 1500 5900 50  0000 C CNN
-F 2 "" H 1500 6050 50  0001 C CNN
-F 3 "" H 1500 6050 50  0001 C CNN
-	1    1500 6050
 	1    0    0    -1
 $EndComp
@@
 	700  5400 700  5300
 Wire Wire Line
-	700  5300 1900 5300
-Wire Wire Line
-	1450 5400 1450 5300
+	1150 5300 1650 5300
 Connection ~ 1450 5300
 Wire Wire Line
 	1650 4900 1550 4900
-Wire Wire Line
-	1550 4900 1550 5300
 Connection ~ 1550 5300
 Wire Wire Line
@@
 Connection ~ 2950 5050
 Wire Wire Line
-	1500 5900 1500 6050
-Wire Wire Line
-	700  5900 3350 5900
+	1500 5900 3350 5900
 Connection ~ 1500 5900
-Wire Wire Line
-	1450 5700 1450 5900
-Connection ~ 1450 5900
 Wire Wire Line
 	2950 5900 2950 5800
@@
 	1650 5450 1900 5450
 Wire Wire Line
-	1650 5450 1650 5300
+	1650 5300 1650 5450
 Connection ~ 1650 5300
 Wire Wire Line
@@
 Connection ~ 6900 650
 Wire Wire Line
-	9900 1550 9900 1250
+	9900 1250 9900 1550
 Connection ~ 9900 1250
 Wire Wire Line
-	9300 1550 9300 1250
+	9300 1250 9300 1550
 Connection ~ 9300 1250
 Wire Wire Line
-	8700 1550 8700 1250
+	8700 1250 8700 1550
 Connection ~ 8700 1250
 Wire Wire Line
-	8100 1550 8100 1250
+	8100 1250 8100 1550
 Connection ~ 8100 1250
 Wire Wire Line
-	7500 1550 7500 1250
+	7500 1250 7500 1550
 Connection ~ 7500 1250
 Wire Wire Line
@@
 Connection ~ 7450 1550
 Wire Wire Line
-	7400 2150 7450 2150
+	7450 2150 7400 2150
 Connection ~ 7450 2150
 Wire Wire Line
-	7400 2750 7450 2750
+	7450 2750 7400 2750
 Connection ~ 7450 2750
 Connection ~ 7450 3350
@@
 	9800 950  9850 950
 Wire Wire Line
-	9850 950  9850 4100
+	9850 950  9850 3350
 Wire Wire Line
 	10400 950  10450 950
@@
 Connection ~ 9250 3350
 Wire Wire Line
-	9800 3350 9850 3350
+	9850 3350 9800 3350
 Connection ~ 9850 3350
 Wire Wire Line
@@
 Connection ~ 1050 5300
 Wire Wire Line
-	5200 6150 5050 6150
-Connection ~ 5200 6150
-Wire Wire Line
-	1050 4950 1050 5300
-Wire Wire Line
-	5200 5650 5200 6150
-Wire Wire Line
 	4700 1900 4700 3250
 Wire Wire Line
@@
 Wire Wire Line
 	5300 5550 4300 5550
-Wire Wire Line
-	5200 5650 6000 5650
-Wire Wire Line
-	6000 5650 6000 4550
 Wire Wire Line
 	6000 4550 5850 4550
@@
 $EndComp
 Wire Wire Line
-	9950 3350 9950 3050
-Wire Wire Line
-	9950 3050 6650 3050
+	9950 3050 9950 3350
+Wire Wire Line
+	6650 3050 9950 3050
 Wire Wire Line
 	3550 1800 4800 1800
 Wire Wire Line
 	3550 1900 4700 1900
+$Comp
+L +3.3V #PWR07
+U 1 1 5AD8D001
+P 700 5300
+F 0 "#PWR07" H 700 5150 50  0001 C CNN
+F 1 "+3.3V" H 700 5440 50  0000 C CNN
+F 2 "" H 700 5300 50  0001 C CNN
+F 3 "" H 700 5300 50  0001 C CNN
+	1    700  5300
+	1    0    0    -1
+$EndComp
+$Comp
+L GND #PWR08
+U 1 1 5AD8D120
+P 700 5900
+F 0 "#PWR08" H 700 5650 50  0001 C CNN
+F 1 "GND" H 700 5750 50  0000 C CNN
+F 2 "" H 700 5900 50  0001 C CNN
+F 3 "" H 700 5900 50  0001 C CNN
+	1    700  5900
+	1    0    0    -1
+$EndComp
 $EndSCHEMATC

Commit message: some changes
Parts:
- added SW1: SW_SPDT, Buttons_Switches_SMD:SW_SPDT_PCM12, symbol SW_SPDT
Connections:
- wire segments 101 -> 100
Changed lines of the file:
@@
 LIBS:switches
 LIBS:mcp1640
+LIBS:interphase-cache
 EELAYER 25 0
 EELAYER END
@@
 	700  5400 700  5300
 Wire Wire Line
-	1150 5300 1650 5300
-Connection ~ 1450 5300
-Wire Wire Line
 	1650 4900 1550 4900
-Connection ~ 1550 5300
 Wire Wire Line
 	1950 4900 2250 4900
@@
 Connection ~ 2950 5050
 Wire Wire Line
-	1500 5900 3350 5900
-Connection ~ 1500 5900
+	1900 5900 3350 5900
 Wire Wire Line
 	2950 5900 2950 5800
@@
 	3350 5900 3350 5600
 Connection ~ 2950 5900
-Wire Wire Line
-	1650 5450 1900 5450
-Wire Wire Line
-	1650 5300 1650 5450
-Connection ~ 1650 5300
 Wire Wire Line
 	10500 650  10500 950
@@
 	9800 950  9850 950
 Wire Wire Line
-	9850 950  9850 3350
+	9850 950  9850 4100
 Wire Wire Line
 	10400 950  10450 950
@@
 Connection ~ 9250 1550
 Connection ~ 700  5900
-Connection ~ 1050 5300
 Wire Wire Line
 	4700 1900 4700 3250
@@
 Wire Wire Line
 	7450 950  7450 3700
-Connection ~ 1150 5300
 Wire Wire Line
 	700  5700 700  5900
@@
 L +3.3V #PWR07
 U 1 1 5AD8D001
-P 700 5300
-F 0 "#PWR07" H 700 5150 50  0001 C CNN
-F 1 "+3.3V" H 700 5440 50  0000 C CNN
-F 2 "" H 700 5300 50  0001 C CNN
-F 3 "" H 700 5300 50  0001 C CNN
-	1    700  5300
+P 800 4900
+F 0 "#PWR07" H 800 4750 50  0001 C CNN
+F 1 "+3.3V" H 800 5040 50  0000 C CNN
+F 2 "" H 800 4900 50  0001 C CNN
+F 3 "" H 800 4900 50  0001 C CNN
+	1    800  4900
 	1    0    0    -1
 $EndComp
@@
 	1    0    0    -1
 $EndComp
+$Comp
+L SW_SPDT SW1
+U 1 1 5ADD68E1
+P 800 5100
+F 0 "SW1" H 800 5270 50  0000 C CNN
+F 1 "SW_SPDT" H 800 4900 50  0000 C CNN
+F 2 "Buttons_Switches_SMD:SW_SPDT_PCM12" H 800 5100 50  0001 C CNN
+F 3 "" H 800 5100 50  0001 C CNN
+	1    800  5100
+	0    1    1    0
+$EndComp
+Wire Wire Line
+	1650 5450 1900 5450
+Connection ~ 1650 5300
+Wire Wire Line
+	1650 5300 1650 5450
 $EndSCHEMATC

Commit message: save previous work
Parts:
- added SW101, SW102: SW_SPDT, Button_Switch_Keyboard:SW_E-Switch_EG1224_SPDT_Angled, symbol SW_SPDT
- added U2: Core51822B, Misc:Core51822(B), symbol Core51822B
- SW1: footprint Buttons_Switches_SMD:SW_SPDT_PCM12 -> Button_Switch_Keyboard:SW_E-Switch_EG1224_SPDT_Angled
Connections:
- net labels removed: +BATT
- wire segments 100 -> 107
